File: Sensors.kicad_sch (KiCad schematic)
At the start: 1 part, among them IC1 ICM-42688-P

Commit message: Update SCH
Parts:
- added C10: 2.2uF, symbol Library:C
- added C11, C13, C14, C15, C18, C19, C20, C42: 0.1uF, symbol Library:C
- added C12: 10nF, symbol Library:C
- added C16, C17: 10uF, symbol Library:C
- added IC4: W25Q256JWPIQ, SON127P600X500X80-9N-D, symbol Library:W25Q256JWPIQ
- added R4: 100K, symbol Library:R
- added R5, R6: 4K7, symbol Library:R
- added R7: 10K, symbol Library:R
- added R8, R9: 75R, symbol Library:R
- added U2: DPS310, SamacSys_Parts:WLGA-8_L2.5-W2.0-P0.65-TR_DPS422, symbol Library:DPS310
- added U3: AT7456E, SamacSys_Parts:TSSOP-28_L9.7-W4.4-P0.65-LS6.4-BL-EP-2, symbol Library:AT7456E
Connections:
- net IMU_MISO: now reaches IC1.1 (AP_SDO_/_AP_AD0)
- net GND: now reaches IC1.10 (RESV_4)
- net GND: now also IC1.11 (RESV_5), IC1.2 (RESV_1), IC1.3 (RESV_2), IC1.6 (GND), IC1.7 (RESV_3), C10.2, C11.2, C12.2, C13.1, C14.1, C15.2, C18.2, C20.2, C42.2, IC4.4 (GND), IC4.9 (EP), R4.2, R9.2, U2.1 (GND), U2.7 (GND), U3.20 (AGND), U3.23 (PGND), U3.29 (EP), U3.4 (DGND)
- net IMU_CS: now reaches IC1.12 (AP_CS)
- net IMU_SCK: now reaches IC1.13 (AP_SCL_/_AP_SCLK)
- net IMU_MOSI: now reaches IC1.14 (AP_SDA_/_AP_SDIO_/_AP_SDI)
- net +3.3V_SENSOR: now reaches IC1.5 (VDDIO)
- net +3.3V_SENSOR: now also IC1.8 (VDD), C10.1, C11.1, C12.1, C13.2, C14.2, R5.2, R6.2, R7.1, U2.6 (VDDIO), U2.8 (VDD)
- net IMU_CLKIN: now reaches IC1.9 (INT2_/_FSYNC_/_CLKIN)
- new net: C16.2, C17.2, R8.1
- new net: R4.1, U2.5 (SDO)
- new net: C17.1, U3.26 (VOUT)
- new net: C19.1, U3.22 (VIN)
- new net: C16.1, U3.25 (SAG)
- new net +3.3V_MCU: C42.1, IC4.3 (~{WP(IO2)}), IC4.7 (~{HOLD_OR_}RESET(IO3)), IC4.8 (VCC)
- new net +5V: C15.1, C18.1, C20.1, U3.19 (RESET#), U3.21 (AVDD), U3.24 (PVDD), U3.3 (DVDD)
- new net BARO_SCL: R6.1, U2.4 (SCK)
- new net BARO_SDA: R5.1, U2.3 (SDI)
- new net FLASH_CS: IC4.1 (~{CS})
- new net FLASH_MISO: IC4.2 (DO(IO1))
- new net FLASH_MOSI: IC4.5 (DI(IO0))
- new net FLASH_SCK: IC4.6 (CLK)
- new net OSC_IN: U3.5 (CLKIN)
- new net OSC_OUT: U3.6 (XFB)
- new net OSD_CS: R7.2, U3.8 (CS#)
- new net OSD_MOSI: U3.11 (SDOUT), U3.9 (SDIN)
- new net OSD_SCK: U3.10 (SCLK)
- new net VRX: C19.2, R9.1
- new net VTX: R8.2
- no-connect marks 0 -> 14
Other:
- moved on the sheet: IC1

Commit message: Update SCH
Parts:
- renumbered C12 to C10, C15 to C11, C13 to C12, C14 to C13, C17 to C14, C16 to C15, C19 to C16, C20 to C17, C11 to C18, C10 to C19, C18 to C20, C42 to C21, IC4 to IC2, R9 to R10, R7 to R5, R5 to R6, R6 to R7, R4 to R8, R8 to R9
Connections:
- net FLASH_CS renamed SPI2_CS
- net FLASH_MISO renamed SPI2_MISO
- net FLASH_MOSI renamed SPI2_MOSI
- net FLASH_SCK renamed SPI2_SCK
- net IMU_CS renamed SPI1_CS
- net IMU_MISO renamed SPI1_MISO
- net IMU_MOSI renamed SPI1_MOSI
- net IMU_SCK renamed SPI1_SCK
- net OSD_CS renamed SPI3_CS
- net OSD_MOSI renamed SPI3_MISO
- net SPI3_MISO: no longer U3.9 (SDIN)
- net OSD_SCK renamed SPI3_SCK
- new net SPI3_MOSI: U3.9 (SDIN)

Commit message: Finished SCH
Parts:
- added C43, C44: 12pF, Capacitor_SMD:C_0402_1005Metric, symbol Library:C
- added Y1: YSX321SL, YSX321SL, symbol SamacSys_Parts:YSX321SL
- C10, C11, C12, C13, C14, C15, C16, C17, C18, C19, C20, C21: footprint (none) -> Capacitor_SMD:C_0402_1005Metric
- R10, R5, R6, R7, R8, R9: footprint (none) -> Resistor_SMD:R_0402_1005Metric
Connections:
- net GND: now also C43.1, C44.2, Y1.2 (GND_1), Y1.4 (GND_2)
- net OSC_IN: now also C43.2, Y1.1 (CRYSTAL_1)
- net OSC_OUT: now also C44.1, Y1.3 (CRYSTAL_2)
Other:
- moved on the sheet: C11, C14, C15, C16, C17, C20, R10, R5, R9, U3

Commit message: Update PCB Layout
Parts:
- added Q2: SS8050, Package_TO_SOT_SMD:SOT-23, symbol Transistor_BJT:SS8050
- added R31: 1K, Resistor_SMD:R_0402_1005Metric, symbol Library:R
Connections:
- net GND: now also Q2.2 (E)
- net +5V renamed VCC_IN
- net BARO_SCL renamed I2C1_SCL
- net BARO_SDA renamed I2C1_SDA
- new net: Q2.1 (B), R31.2
- new net BEEPER: R31.1
- new net BEEPER-: Q2.3 (C)
