File: Power.kicad_sch (KiCad schematic)
At the start: 43 parts, among them IC2 LP2992IM5-3.3, IC3 LP2992IM5-3.3, U4 MP9943AGQ-Z, U5 MP9943AGQ-Z

Commit message: Update SCH
Parts:
- renumbered C35 to C23, C38 to C24, C41 to C25, C21 to C26, C23 to C27, C24 to C28, C26 to C29, C36 to C30, C37 to C31, C39 to C32, C40 to C33, C25 to C34, C27 to C35, C28 to C36, C29 to C37, C30 to C38, C31 to C39, C32 to C40, C33 to C41, C34 to C42, IC2 to IC3, IC3 to IC4, R15 to R11, R13 to R12, R14 to R13, R10 to R14, R21 to R15, R22 to R16, R12 to R17, R16 to R18, R17 to R19, R18 to R20, R19 to R21, R20 to R22

Commit message: Finished SCH
Parts:
- added C45, C46: 22uF, Capacitor_SMD:C_0805_2012Metric, symbol Library:C
- C22, C26, C30, C32, C36, C37: footprint (none) -> Capacitor_SMD:C_0402_1005Metric
- C23, C24, C31, C33: footprint (none) -> Capacitor_SMD:C_0603_1608Metric
- C25: value 100nF -> 0.1uF; footprint (none) -> Capacitor_SMD:C_0402_1005Metric
- C27, C28, C29, C34, C35, C38, C39, C40, C41, C42: footprint (none) -> Capacitor_SMD:C_0805_2012Metric
- F1: footprint (none) -> Resistor_SMD:R_1206_3216Metric
- L2, L3: footprint (none) -> Inductor_SMD:L_APV_APH0530
- R11, R12, R13, R14, R15, R16, R17, R18, R19, R20, R21, R22: footprint (none) -> Resistor_SMD:R_0402_1005Metric
Connections:
- net GND: now also C45.2, C46.2
- net VCC_10V: now also C46.1
- net VCC_5V: now also C45.1
Other:
- moved on the sheet: C27, C28, C29, C34, C35, C38, C39, C40, C41, C42, R17, R22

Commit message: Update PCB Layout
Parts:
- added C48: 1uF, Capacitor_SMD:C_0603_1608Metric, symbol Library:C
- added C49: 10nF, Capacitor_SMD:C_0402_1005Metric, symbol Library:C
- added C50: 2.2uF, Capacitor_SMD:C_0603_1608Metric, symbol Library:C
- added D6: LED, LED_SMD:LED_0603_1608Metric, symbol Device:LED
- added IC5: LP2992IM5-3.3, SOT95P280X145-5N, symbol Library:LP2992IM5-3.3
- added R32: 100R, Resistor_SMD:R_0402_1005Metric, symbol Library:R
Connections:
- net VCC_5V_IN is gone; now on net VCC_5V: C23.1, C24.1, IC3.1 (IN), IC3.3 (ON/~{OFF}), IC4.1 (IN), IC4.3 (ON/~{OFF})
- net +3.3V_MCU: now also R32.2
- net +3.3V_SENSOR: now also C50.1, IC5.5 (OUT)
- net GND: now also C48.2, C49.2, C50.2, D6.1 (K), IC5.2 (GND)
- net VCC_5V: now also C48.1, IC5.1 (IN), IC5.3 (ON/~{OFF})
- new net: C49.1, IC5.4 (BYPASS)
- new net: D6.2 (A), R32.1

Commit message: Finished PCB V1.0
Connections:
- net +3.3V_SENSOR: no longer C50.1, IC5.5 (OUT)
- net VCC_5V: no longer C23.1, C24.1, C48.1, IC3.1 (IN), IC3.3 (ON/~{OFF}), IC4.1 (IN), IC4.3 (ON/~{OFF}), IC5.1 (IN), IC5.3 (ON/~{OFF})
- net VCC_IN: now also C23.1, C24.1, C48.1, IC3.1 (IN), IC3.3 (ON/~{OFF}), IC4.1 (IN), IC4.3 (ON/~{OFF}), IC5.1 (IN), IC5.3 (ON/~{OFF})
- net EN renamed EN1
- net EN1: no longer R22.1, U5.3 (EN/SYNC)
- new net +3.3V_PREP: C50.1, IC5.5 (OUT)
- new net EN2: R22.1, U5.3 (EN/SYNC)
Changed lines of the file:
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@@
 	(wire
 		(pts
-			(xy 157.48 40.64) (xy 160.02 40.64)
+			(xy 154.94 40.64) (xy 160.02 40.64)
 		)
 		(stroke
@@
 	(wire
 		(pts
-			(xy 45.72 40.64) (xy 48.26 40.64)
+			(xy 41.91 40.64) (xy 48.26 40.64)
 		)
 		(stroke
@@
 		)
 	)
-	(label "EN"
+	(label "EN2"
 		(at 205.74 25.4 0)
 		(effects
@@
 		)
 	)
-	(label "EN"
-		(at 93.98 25.4 0)
+	(label "EN2"
+		(at 154.94 40.64 0)
 		(effects
 			(font
@@
 		)
 	)
-	(label "EN"
-		(at 45.72 40.64 0)
+	(label "EN1"
+		(at 41.91 40.64 0)
 		(effects
 			(font
@@
 		)
 	)
-	(label "EN"
-		(at 157.48 40.64 0)
+	(label "EN1"
+		(at 93.98 25.4 0)
 		(effects
 			(font
@@
 	)
 	(symbol
-		(lib_id "power:VCC")
-		(at 35.56 139.7 90)
-		(unit 1)
-		(exclude_from_sim no)
-		(in_bom yes)
-		(on_board yes)
-		(dnp no)
-		(fields_autoplaced yes)
-		(property "Reference" "#PWR044"
-			(at 39.37 139.7 0)
-			(effects
-				(font
-					(size 1.27 1.27)
-				)
-				(hide yes)
-			)
-		)
-		(property "Value" "VCC_5V"
-			(at 31.75 139.6999 90)
-			(effects
-				(font
-					(size 1.27 1.27)
-				)
-				(justify left)
-			)
-		)
-		(property "Footprint" ""
-			(at 35.56 139.7 0)
-			(effects
-				(font
-					(size 1.27 1.27)
-				)
-				(hide yes)
-			)
-		)
-		(property "Datasheet" ""
-			(at 35.56 139.7 0)
-			(effects
-				(font
-					(size 1.27 1.27)
-				)
-				(hide yes)
-			)
-		)
-		(property "Description" "Power symbol creates a global label with name \"VCC\""
-			(at 35.56 139.7 0)
-			(effects
-				(font
-					(size 1.27 1.27)
-				)
-				(hide yes)
-			)
-		)
-		(pin "1"
-		)
-		(instances
-			(project "NekoPurrTech_Skylark"
-				(path "/0bcb4a44-4fa7-4976-a48b-273b8974ffc7/2cb43c0a-747a-47ba-9a71-a2b1eea6abcf"
-					(reference "#PWR044")
-					(unit 1)
-				)
-			)
-		)
-	)
-	(symbol
 		(lib_id "power:GND")
 		(at 96.52 124.46 0)
@@
 		(dnp no)
 		(fields_autoplaced yes)
-		(property "Reference" "#PWR0137"
+		(property "Reference" "#PWR0139"
 			(at 39.37 111.76 0)
 			(effects
@@
 			)
 		)
-		(property "Value" "VCC_5V"
+		(property "Value" "VCC_IN"
 			(at 31.75 111.7599 90)
 			(effects
@@
 			(project "NekoPurrTech_Skylark"
 				(path "/0bcb4a44-4fa7-4976-a48b-273b8974ffc7/2cb43c0a-747a-47ba-9a71-a2b1eea6abcf"
-					(reference "#PWR0137")
+					(reference "#PWR0139")
 					(unit 1)
 				)
@@
 	)
 	(symbol
-		(lib_id "power:VCC")
-		(at 35.56 81.28 90)
-		(unit 1)
-		(exclude_from_sim no)
-		(in_bom yes)
-		(on_board yes)
-		(dnp no)
-		(fields_autoplaced yes)
-		(property "Reference" "#PWR0136"
-			(at 39.37 81.28 0)
-			(effects
-				(font
-					(size 1.27 1.27)
-				)
-				(hide yes)
-			)
-		)
-		(property "Value" "VCC_5V"
-			(at 31.75 81.2799 90)
-			(effects
-				(font
-					(size 1.27 1.27)
-				)
-				(justify left)
-			)
-		)
-		(property "Footprint" ""
-			(at 35.56 81.28 0)
-			(effects
-				(font
-					(size 1.27 1.27)
-				)
-				(hide yes)
-			)
-		)
-		(property "Datasheet" ""
-			(at 35.56 81.28 0)
-			(effects
-				(font
-					(size 1.27 1.27)
-				)
-				(hide yes)
-			)
-		)
-		(property "Description" "Power symbol creates a global label with name \"VCC\""
-			(at 35.56 81.28 0)
-			(effects
-				(font
-					(size 1.27 1.27)
-				)
-				(hide yes)
-			)
-		)
-		(pin "1"
-		)
-		(instances
-			(project "NekoPurrTech_Skylark"
-				(path "/0bcb4a44-4fa7-4976-a48b-273b8974ffc7/2cb43c0a-747a-47ba-9a71-a2b1eea6abcf"
-					(reference "#PWR0136")
-					(unit 1)
-				)
-			)
-		)
-	)
-	(symbol
 		(lib_id "Library:R")
 		(at 176.53 125.73 90)
@@
 			)
 		)
-		(property "Value" "+3.3V_SENSOR"
+		(property "Value" "+3.3V_PREP"
 			(at 107.95 142.2399 90)
 			(effects
@@
 	)
 	(symbol
+		(lib_id "power:VCC")
+		(at 35.56 139.7 90)
+		(unit 1)
+		(exclude_from_sim no)
+		(in_bom yes)
+		(on_board yes)
+		(dnp no)
+		(fields_autoplaced yes)
+		(property "Reference" "#PWR0136"
+			(at 39.37 139.7 0)
+			(effects
+				(font
+					(size 1.27 1.27)
+				)
+				(hide yes)
+			)
+		)
+		(property "Value" "VCC_IN"
+			(at 31.75 139.6999 90)
+			(effects
+				(font
+					(size 1.27 1.27)
+				)
+				(justify left)
+			)
+		)
+		(property "Footprint" ""
+			(at 35.56 139.7 0)
+			(effects
+				(font
+					(size 1.27 1.27)
+				)
+				(hide yes)
+			)
+		)
+		(property "Datasheet" ""
+			(at 35.56 139.7 0)
+			(effects
+				(font
+					(size 1.27 1.27)
+				)
+				(hide yes)
+			)
+		)
+		(property "Description" "Power symbol creates a global label with name \"VCC\""
+			(at 35.56 139.7 0)
+			(effects
+				(font
+					(size 1.27 1.27)
+				)
+				(hide yes)
+			)
+		)
+		(pin "1"
+		)
+		(instances
+			(project "NekoPurrTech_Skylark"
+				(path "/0bcb4a44-4fa7-4976-a48b-273b8974ffc7/2cb43c0a-747a-47ba-9a71-a2b1eea6abcf"
+					(reference "#PWR0136")
+					(unit 1)
+				)
+			)
+		)
+	)
+	(symbol
 		(lib_id "power:GND")
 		(at 80.01 49.53 0)
@@
 					(unit 1)
 				)
+			)
+		)
+	)
+	(symbol
+		(lib_id "power:VCC")
+		(at 35.56 81.28 90)
+		(unit 1)
+		(exclude_from_sim no)
+		(in_bom yes)
+		(on_board yes)
+		(dnp no)
+		(fields_autoplaced yes)
+		(property "Reference" "#PWR044"
+			(at 39.37 81.28 0)
+			(effects
+				(font
+					(size 1.27 1.27)
+				)
+				(hide yes)
+			)
+		)
+		(property "Value" "VCC_IN"
+			(at 31.75 81.2799 90)
+			(effects
+				(font
+					(size 1.27 1.27)
+				)
+				(justify left)
+			)
+		)
+		(property "Footprint" ""
+			(at 35.56 81.28 0)
+			(effects
+				(font
+					(size 1.27 1.27)
+				)
+				(hide yes)
+			)
+		)
+		(property "Datasheet" ""
+			(at 35.56 81.28 0)
+			(effects
+				(font
+					(size 1.27 1.27)
+				)
+				(hide yes)
+			)
+		)
+		(property "Description" "Power symbol creates a global label with name \"VCC\""
+			(at 35.56 81.28 0)
+			(effects
+				(font
+					(size 1.27 1.27)
+				)
+				(hide yes)
+			)
+		)
+		(pin "1"
+		)
+		(instances
+			(project "NekoPurrTech_Skylark"
+				(path "/0bcb4a44-4fa7-4976-a48b-273b8974ffc7/2cb43c0a-747a-47ba-9a71-a2b1eea6abcf"
+					(reference "#PWR044")
+					(unit 1)
+				)
