File: NekoPurrTech_Skylark.kicad_pcb (KiCad board)
At the start: 2 copper layers, 6 parts, among them IC1 ICM-42688-P, U1 STM32F405RGTx

Commit message: Update SCH
Parts:
- added D1: SMAJ30CA, Library:D_SMA, F.Cu at (107.0, 49.5)
- added D2: 1N5819WS, Library:D_SOD-323, F.Cu at (105.2, 53.2)
- added D3: 1N5819WS, Library:D_SOD-323, F.Cu at (105.2, 56.2)
- added IC2: LP2992IM5-3.3, Library:SOT95P280X145-5N, F.Cu at (71.7, 80.7)
- added IC3: LP2992IM5-3.3, Library:SOT95P280X145-5N, F.Cu at (75.9, 80.8)
- added IC4: W25Q256JWPIQ, Library:SON127P600X500X80-9N-D, F.Cu at (128.7, 80.9)
- added J1: DJI_VTX, Library:JST_SH_SM06B-SRSS-TB_1x06-1MP_P1.00mm_Horizontal, F.Cu at (145.9, 89.6)
- added J2: Motor, Library:JST_SH_SM08B-SRSS-TB_1x08-1MP_P1.00mm_Horizontal, F.Cu at (171.1, 99.2)
- added J3: GPS, Library:JST_SH_SM06B-SRSS-TB_1x06-1MP_P1.00mm_Horizontal, F.Cu at (145.9, 101.5)
- added J4: CRSF_Receiver, Library:JST_SH_SM04B-SRSS-TB_1x04-1MP_P1.00mm_Horizontal, F.Cu at (145.9, 101.5)
- added J5: Analog_Camera, Library:JST_SH_SM03B-SRSS-TB_1x03-1MP_P1.00mm_Horizontal, F.Cu at (171.2, 88.3)
- added J6: Analog_VTX, Library:JST_SH_SM05B-SRSS-TB_1x05-1MP_P1.00mm_Horizontal, F.Cu at (145.8, 89.6)
- added U2: DPS310, Library:WLGA-8_L2.5-W2.0-P0.65-TR_DPS422, F.Cu at (87.0, 80.9)
- added U3: AT7456E, Library:TSSOP-28_L9.7-W4.4-P0.65-LS6.4-BL-EP-2, F.Cu at (94.9, 70.0)
- added U4: MP9943AGQ-Z, Library:QFN-8_L3.0-W3.0-P0.65, F.Cu at (76.0, 73.2)
- added U5: MP9943AGQ-Z, Library:QFN-8_L3.0-W3.0-P0.65, F.Cu at (71.4, 73.2)
- moved U1 158.7 mm to (216.6, 108.4)
- moved IC1 23.2 mm to (83.3, 80.9)
Connections:
- IC1 pad 1: unconnected-(IC1-AP_SDO_/_AP_AD0-Pad1) -> IMU_MISO
- IC1 pad 10: unconnected-(IC1-RESV_4-Pad10) -> GND
- IC1 pad 11: unconnected-(IC1-RESV_5-Pad11) -> GND
- IC1 pad 12: unconnected-(IC1-AP_CS-Pad12) -> IMU_CS
- IC1 pad 13: unconnected-(IC1-AP_SCL_/_AP_SCLK-Pad13) -> IMU_SCK
- IC1 pad 14: unconnected-(IC1-AP_SDA_/_AP_SDIO_/_AP_SDI-Pad14) -> IMU_MOSI
- IC1 pad 2: unconnected-(IC1-RESV_1-Pad2) -> GND
- IC1 pad 3: unconnected-(IC1-RESV_2-Pad3) -> GND
- IC1 pad 5: unconnected-(IC1-VDDIO-Pad5) -> +3.3V_SENSOR
- IC1 pad 6: unconnected-(IC1-GND-Pad6) -> GND
- IC1 pad 7: unconnected-(IC1-RESV_3-Pad7) -> GND
- IC1 pad 8: unconnected-(IC1-VDD-Pad8) -> +3.3V_SENSOR
- IC1 pad 9: unconnected-(IC1-INT2_/_FSYNC_/_CLKIN-Pad9) -> IMU_CLKIN
Other:
- board outline added: 40 x 40 mm

Commit message: Update SCH
Parts:
- D1: footprint Library:D_SMA -> Diode_SMD:D_SMA
- D2, D3: footprint Library:D_SOD-323 -> Diode_SMD:D_SOD-323
- IC2: renamed from IC4; moved to B.Cu
- J1: renamed from J2; footprint Library:JST_SH_SM08B-SRSS-TB_1x08-1MP_P1.00mm_Horizontal -> Connector_JST:JST_SH_SM08B-SRSS-TB_1x08-1MP_P1.00mm_Horizontal; moved to B.Cu
- J2: renamed from J1; footprint Library:JST_SH_SM06B-SRSS-TB_1x06-1MP_P1.00mm_Horizontal -> Connector_JST:JST_SH_SM06B-SRSS-TB_1x06-1MP_P1.00mm_Horizontal; moved to B.Cu
- J3: footprint Library:JST_SH_SM06B-SRSS-TB_1x06-1MP_P1.00mm_Horizontal -> Connector_JST:JST_SH_SM06B-SRSS-TB_1x06-1MP_P1.00mm_Horizontal; moved to B.Cu
- J4: footprint Library:JST_SH_SM04B-SRSS-TB_1x04-1MP_P1.00mm_Horizontal -> Connector_JST:JST_SH_SM04B-SRSS-TB_1x04-1MP_P1.00mm_Horizontal; moved to B.Cu
- J5: footprint Library:JST_SH_SM03B-SRSS-TB_1x03-1MP_P1.00mm_Horizontal -> Connector_JST:JST_SH_SM03B-SRSS-TB_1x03-1MP_P1.00mm_Horizontal; moved to B.Cu
- J6: footprint Library:JST_SH_SM05B-SRSS-TB_1x05-1MP_P1.00mm_Horizontal -> Connector_JST:JST_SH_SM05B-SRSS-TB_1x05-1MP_P1.00mm_Horizontal; moved to B.Cu
- R2: renamed from R11; footprint Library:R_0603_1608Metric -> Resistor_SMD:R_0603_1608Metric
- R3: footprint Library:R_0603_1608Metric -> Resistor_SMD:R_0603_1608Metric
- U1: footprint Library:LQFP-64_10x10mm_P0.5mm -> Package_QFP:LQFP-64_10x10mm_P0.5mm
- U3: moved to B.Cu
- moved U1 195.1 mm to (31.9, 45.5), turned to 180 degrees
- moved J5 156.6 mm to (26.9, 27.4), turned to 0 degrees
- moved J1 152.8 mm to (36.2, 27.4), turned to 0 degrees
- moved J3 125.0 mm to (28.7, 57.9), turned to 180 degrees
- moved J4 124.3 mm to (46.0, 27.4), turned to 0 degrees
- moved J2 113.2 mm to (37.2, 57.9), turned to 180 degrees
- moved J6 105.5 mm to (45.1, 57.9), turned to 180 degrees
- moved IC2 94.6 mm to (45.4, 36.0), turned to 90 degrees
- moved IC1 70.5 mm to (30.9, 33.9)
- moved U2 69.1 mm to (36.4, 33.9), turned to -90 degrees
- moved U3 54.6 mm to (45.3, 47.1), turned to -90 degrees
- moved R4 36.5 mm to (40.1, 46.9), turned to 90 degrees
- renumbered IC2 to IC3, IC3 to IC4, R2 to R4
Connections:
- IC1 pad 1: IMU_MISO -> SPI1_MISO
- IC1 pad 12: IMU_CS -> SPI1_CS
- IC1 pad 13: IMU_SCK -> SPI1_SCK
- IC1 pad 14: IMU_MOSI -> SPI1_MOSI
- IC2 pad 1: FLASH_CS -> SPI2_CS
- IC2 pad 2: FLASH_MISO -> SPI2_MISO
- IC2 pad 5: FLASH_MOSI -> SPI2_MOSI
- IC2 pad 6: FLASH_SCK -> SPI2_SCK
- IC3 pad 4: unconnected-(C36-Pad1) -> Net-(IC3-BYPASS)
- U1 pad 10: unconnected-(U1-PC2-Pad10) -> SPI2_MISO
- U1 pad 11: unconnected-(U1-PC3-Pad11) -> SPI2_MOSI
- U1 pad 20: unconnected-(U1-PA4-Pad20) -> SPI1_CS
- U1 pad 21: unconnected-(U1-PA5-Pad21) -> SPI1_SCK
- U1 pad 22: unconnected-(U1-PA6-Pad22) -> SPI1_MISO
- U1 pad 23: unconnected-(U1-PA7-Pad23) -> SPI1_MOSI
- U1 pad 33: unconnected-(U1-PB12-Pad33) -> SPI2_CS
- U1 pad 34: unconnected-(U1-PB13-Pad34) -> SPI2_SCK
- U1 pad 50: unconnected-(U1-PA15-Pad50) -> SPI3_CS
- U1 pad 55: unconnected-(U1-PB3-Pad55) -> SPI3_SCK
- U1 pad 56: unconnected-(U1-PB4-Pad56) -> SPI3_MISO
- U1 pad 57: unconnected-(U1-PB5-Pad57) -> SPI3_MOSI
- U1 pad 58: unconnected-(U1-PB6-Pad58) -> BARO_SCL
- U1 pad 59: unconnected-(U1-PB7-Pad59) -> BARO_SDA
- U3 pad 10: OSD_SCK -> SPI3_SCK
- U3 pad 11: OSD_MOSI -> SPI3_MISO
- U3 pad 8: OSD_CS -> SPI3_CS
- U3 pad 9: OSD_MOSI -> SPI3_MOSI
- U4 pad 1: unconnected-(R13-Pad1) -> Net-(U4-FB)
- U4 pad 2: unconnected-(C22-Pad1) -> Net-(U4-VCC)
- U4 pad 4: (no net) -> Net-(U4-BST)
- U4 pad 6: unconnected-(C21-Pad2) -> Net-(U4-SW)
- U4 pad 8: (no net) -> unconnected-(U4-PG-Pad8)
Other:
- board size 40 x 40 mm -> 36.5 x 36.5 mm

Commit message: Finished SCH
Parts:
- removed J6: Analog_VTX, Connector_JST:JST_SH_SM05B-SRSS-TB_1x05-1MP_P1.00mm_Horizontal
- added C1: 0.1uF, Capacitor_SMD:C_0402_1005Metric, F.Cu at (34.9, 50.8)
- added C10: 10nF, Capacitor_SMD:C_0402_1005Metric, F.Cu at (27.4, 32.8)
- added C11: 0.1uF, Capacitor_SMD:C_0402_1005Metric, B.Cu at (29.6, 52.5)
- added C12: 0.1uF, Capacitor_SMD:C_0402_1005Metric, F.Cu at (34.9, 30.5)
- added C13: 0.1uF, Capacitor_SMD:C_0402_1005Metric, F.Cu at (30.8, 30.5)
- added C14: 10uF, Capacitor_SMD:C_0402_1005Metric, B.Cu at (32.2, 42.9)
- added C15: 10uF, Capacitor_SMD:C_0402_1005Metric, B.Cu at (31.2, 42.9)
- added C16: 0.1uF, Capacitor_SMD:C_0402_1005Metric, B.Cu at (28.3, 42.9)
- added C17: 0.1uF, Capacitor_SMD:C_0402_1005Metric, B.Cu at (29.3, 42.9)
- added C18: 0.1uF, Capacitor_SMD:C_0402_1005Metric, F.Cu at (28.4, 32.8)
- added C19: 2.2uF, Capacitor_SMD:C_0402_1005Metric, F.Cu at (29.5, 32.8)
- added C2: 0.1uF, Capacitor_SMD:C_0402_1005Metric, F.Cu at (22.9, 46.6)
- added C20: 0.1uF, Capacitor_SMD:C_0402_1005Metric, F.Cu at (8.10, 48.7)
- added C21: 0.1uF, Capacitor_SMD:C_0402_1005Metric, B.Cu at (49.6, 51.6)
- added C22: 0.1uF, Capacitor_SMD:C_0402_1005Metric, B.Cu at (46.6, 31.4)
- added C23: 1uF, Capacitor_SMD:C_0603_1608Metric, B.Cu at (34.6, 41.7)
- added C24: 1uF, Capacitor_SMD:C_0603_1608Metric, B.Cu at (20.2, 41.9)
- added C25: 0.1uF, Capacitor_SMD:C_0402_1005Metric, B.Cu at (39.6, 20.3)
- added C26: 0.1uF, Capacitor_SMD:C_0402_1005Metric, B.Cu at (40.9, 31.4)
- added C27: 1uF/50V, Capacitor_SMD:C_0805_2012Metric, B.Cu at (35.6, 33.7)
- added C28: 10uF/50V, Capacitor_SMD:C_0805_2012Metric, B.Cu at (37.6, 33.7)
- added C29: 22uF, Capacitor_SMD:C_0805_2012Metric, B.Cu at (37.6, 37.6)
- added C3: 0.1uF, Capacitor_SMD:C_0402_1005Metric, F.Cu at (33.9, 35.0)
- added C30: 10nF, Capacitor_SMD:C_0402_1005Metric, B.Cu at (14.7, 44.9)
- added C31: 2.2uF, Capacitor_SMD:C_0603_1608Metric, B.Cu at (39.9, 41.8)
- added C32: 10nF, Capacitor_SMD:C_0402_1005Metric, B.Cu at (15.1, 41.4)
- added C33: 2.2uF, Capacitor_SMD:C_0603_1608Metric, B.Cu at (25.7, 41.8)
- added C34: 10uF/50V, Capacitor_SMD:C_0805_2012Metric, B.Cu at (39.5, 33.7)
- added C35: 22uF, Capacitor_SMD:C_0805_2012Metric, B.Cu at (39.5, 37.6)
- added C36: 0.1uF, Capacitor_SMD:C_0402_1005Metric, B.Cu at (32.4, 31.4)
- added C37: 0.1uF, Capacitor_SMD:C_0402_1005Metric, B.Cu at (26.7, 31.4)
- added C38: 1uF/50V, Capacitor_SMD:C_0805_2012Metric, B.Cu at (23.3, 33.7)
- added C39: 10uF/50V, Capacitor_SMD:C_0805_2012Metric, B.Cu at (25.3, 33.7)
- added C4: 0.1uF, Capacitor_SMD:C_0402_1005Metric, F.Cu at (27.4, 35.0)
- added C40: 22uF, Capacitor_SMD:C_0805_2012Metric, B.Cu at (21.4, 37.6)
- added C41: 10uF/50V, Capacitor_SMD:C_0805_2012Metric, B.Cu at (21.4, 33.7)
- added C42: 22uF, Capacitor_SMD:C_0805_2012Metric, B.Cu at (25.3, 37.6)
- added C43: 12pF, Capacitor_SMD:C_0402_1005Metric, B.Cu at (37.1, 50.6)
- added C44: 12pF, Capacitor_SMD:C_0402_1005Metric, B.Cu at (37.2, 45.8)
- added C45: 22uF, Capacitor_SMD:C_0805_2012Metric, B.Cu at (35.6, 37.6)
- added C46: 22uF, Capacitor_SMD:C_0805_2012Metric, B.Cu at (23.3, 37.6)
- added C5: 0.1uF, Capacitor_SMD:C_0402_1005Metric, F.Cu at (39.7, 40.8)
- added C6: 1uF, Capacitor_SMD:C_0402_1005Metric, F.Cu at (39.7, 41.7)
- added C7: 0.1uF, Capacitor_SMD:C_0402_1005Metric, F.Cu at (41.5, 40.8)
- added C8: 2.2uF, Capacitor_SMD:C_0402_1005Metric, F.Cu at (28.4, 35.1)
- added C9: 2.2uF, Capacitor_SMD:C_0402_1005Metric, F.Cu at (22.9, 45.5)
- added D4: LED, LED_SMD:LED_0603_1608Metric, F.Cu at (47.8, 50.0)
- added D5: LED, LED_SMD:LED_0603_1608Metric, F.Cu at (47.8, 52.6)
- added F1: 1206_3A, Resistor_SMD:R_1206_3216Metric, B.Cu at (34.5, 29.3)
- added H1: MountingHole_Pad, MountingHole:MountingHole_3.2mm_M3_DIN965_Pad, F.Cu at (21.8, 27.4)
- added H2: MountingHole_Pad, MountingHole:MountingHole_3.2mm_M3_DIN965_Pad, F.Cu at (52.3, 27.4)
- added H3: MountingHole_Pad, MountingHole:MountingHole_3.2mm_M3_DIN965_Pad, F.Cu at (52.3, 57.9)
- added H4: MountingHole_Pad, MountingHole:MountingHole_3.2mm_M3_DIN965_Pad, F.Cu at (21.8, 57.9)
- added J7: USB_C_Receptacle, SamacSys_Parts:USB-C_halfboard, F.Cu at (55.3, 45.0)
- added L1: L, Inductor_SMD:L_0603_1608Metric, F.Cu at (83.5, 44.1)
- added L2: 10uH, Inductor_SMD:L_APV_APH0530, B.Cu at (43.8, 38.2)
- added L3: 10uH, Inductor_SMD:L_APV_APH0530, B.Cu at (29.5, 38.2)
- added R1: 10K, Resistor_SMD:R_0402_1005Metric, F.Cu at (41.5, 41.6)
- added R10: 75R, Resistor_SMD:R_0402_1005Metric, B.Cu at (27.4, 42.9)
- added R11: 41.2K, Resistor_SMD:R_0402_1005Metric, B.Cu at (47.5, 35.1)
- added R12: 51K, Resistor_SMD:R_0402_1005Metric, B.Cu at (46.5, 33.1)
- added R13: 7.68K, Resistor_SMD:R_0402_1005Metric, B.Cu at (47.5, 33.1)
- added R14: 20R, Resistor_SMD:R_0402_1005Metric, B.Cu at (42.8, 31.4)
- added R15: 10K, Resistor_SMD:R_0402_1005Metric, B.Cu at (37.7, 20.3)
- added R16: 1K, Resistor_SMD:R_0402_1005Metric, B.Cu at (38.6, 20.3)
- added R17: 1M, Resistor_SMD:R_0402_1005Metric, B.Cu at (44.7, 31.4)
- added R18: 41.2K, Resistor_SMD:R_0402_1005Metric, B.Cu at (33.3, 35.1)
- added R19: 51K, Resistor_SMD:R_0402_1005Metric, B.Cu at (32.3, 33.1)
- added R20: 3.4K, Resistor_SMD:R_0402_1005Metric, B.Cu at (33.3, 33.1)
- added R21: 20R, Resistor_SMD:R_0402_1005Metric, B.Cu at (28.6, 31.4)
- added R22: 1M, Resistor_SMD:R_0402_1005Metric, B.Cu at (30.5, 31.4)
- added R23: 5K1, Resistor_SMD:R_0402_1005Metric, F.Cu at (46.0, 41.1)
- added R24: 5K1, Resistor_SMD:R_0402_1005Metric, F.Cu at (46.0, 38.1)
- added R25: 100R, Resistor_SMD:R_0402_1005Metric, F.Cu at (50.2, 50.2)
- added R26: 100R, Resistor_SMD:R_0402_1005Metric, F.Cu at (50.2, 52.2)
- added R27: 22R, Resistor_SMD:R_0402_1005Metric, F.Cu at (46.0, 40.1)
- added R28: 22R, Resistor_SMD:R_0402_1005Metric, F.Cu at (46.0, 39.1)
- added R5: 10K, Resistor_SMD:R_0402_1005Metric, B.Cu at (32.1, 52.5)
- added R6: 4K7, Resistor_SMD:R_0402_1005Metric, F.Cu at (32.6, 32.8)
- added R7: 4K7, Resistor_SMD:R_0402_1005Metric, F.Cu at (31.6, 32.8)
- added R8: 100K, Resistor_SMD:R_0402_1005Metric, F.Cu at (33.6, 32.8)
- added R9: 75R, Resistor_SMD:R_0402_1005Metric, B.Cu at (30.2, 42.9)
- added U6: 74LVC1G04, Package_TO_SOT_SMD:SOT-23-5, B.Cu at (21.6, 48.1)
- added U7: USBLC6-2P6, Package_TO_SOT_SMD:SOT-666, F.Cu at (45.6, 44.1)
- added Y1: YSX321SL, SamacSys_Parts:YSX321SL, B.Cu at (37.2, 48.2)
- D1, D2, D3, IC3, IC4: moved to B.Cu
- R2, R3: footprint Resistor_SMD:R_0603_1608Metric -> Resistor_SMD:R_0402_1005Metric
- U2: footprint Library:WLGA-8_L2.5-W2.0-P0.65-TR_DPS422 -> SamacSys_Parts:WLGA-8_L2.5-W2.0-P0.65-TR_DPS422
- U3: footprint Library:TSSOP-28_L9.7-W4.4-P0.65-LS6.4-BL-EP-2 -> SamacSys_Parts:TSSOP-28_L9.7-W4.4-P0.65-LS6.4-BL-EP-2
- U4, U5: footprint Library:QFN-8_L3.0-W3.0-P0.65 -> SamacSys_Parts:QFN-8_L3.0-W3.0-P0.65; moved to B.Cu
- moved D1 76.1 mm to (34.5, 26.3)
- moved IC4 65.7 mm to (23.0, 41.8)
- moved D2 64.1 mm to (41.8, 43.6), turned to -90 degrees
- moved D3 61.7 mm to (44.8, 43.6), turned to -90 degrees
- moved U5 57.5 mm to (29.6, 33.7), turned to -90 degrees
- moved IC3 52.0 mm to (37.2, 41.7)
- moved U4 50.9 mm to (43.8, 33.7), turned to -90 degrees
- moved J4 31.8 mm to (37.0, 57.9), turned to 180 degrees
- moved S1 23.7 mm to (73.0, 53.8)
- moved U3 16.4 mm to (28.9, 48.1), turned to 180 degrees
- moved R3 15.5 mm to (60.5, 66.8)
- moved R2 15.5 mm to (60.5, 69.3)
- moved IC2 14.4 mm to (45.5, 50.4), turned to 180 degrees
- moved J2 7.69 mm to (44.9, 57.9)
- moved J1 7.67 mm to (43.9, 27.4)
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Connections:
- J2 pad 6: SBUS -> /Connectors/SBUS_IN
- U1 pad 14: unconnected-(U1-PA0-Pad14) -> USART4_TX
- U1 pad 15: unconnected-(U1-PA1-Pad15) -> USART4_RX
- U1 pad 16: unconnected-(U1-PA2-Pad16) -> USART2_TX
- U1 pad 17: unconnected-(U1-PA3-Pad17) -> USART2_RX
- U1 pad 2: unconnected-(U1-PC13-Pad2) -> /MCU_Core/LED1
- U1 pad 25: unconnected-(U1-PC5-Pad25) -> ADC_RSSI
- U1 pad 26: unconnected-(U1-PB0-Pad26) -> MOTOR3
- U1 pad 27: unconnected-(U1-PB1-Pad27) -> MOTOR4
- U1 pad 29: unconnected-(U1-PB10-Pad29) -> MOTOR1
- U1 pad 3: unconnected-(U1-PC14-Pad3) -> /MCU_Core/LED2
- U1 pad 30: unconnected-(U1-PB11-Pad30) -> MOTOR2
- U1 pad 36: unconnected-(U1-PB15-Pad36) -> GYRO_CLK
- U1 pad 37: unconnected-(U1-PC6-Pad37) -> USART6_TX
- U1 pad 38: unconnected-(U1-PC7-Pad38) -> USART6_RX
- U1 pad 39: unconnected-(U1-PC8-Pad39) -> LED_STRIP
- U1 pad 40: unconnected-(U1-PC9-Pad40) -> I2C3_SDA
- U1 pad 41: unconnected-(U1-PA8-Pad41) -> I2C3_SCL
- U1 pad 43: unconnected-(U1-PA10-Pad43) -> USART1_RX
- U1 pad 44: unconnected-(U1-PA11-Pad44) -> USB_DN
- U1 pad 45: unconnected-(U1-PA12-Pad45) -> USB_DP
- U1 pad 46: unconnected-(U1-PA13-Pad46) -> SWDIO
- U1 pad 49: unconnected-(U1-PA14-Pad49) -> SWCLK
- U1 pad 51: unconnected-(U1-PC10-Pad51) -> USART3_TX
- U1 pad 52: unconnected-(U1-PC11-Pad52) -> USART3_RX
- U1 pad 54: unconnected-(U1-PD2-Pad54) -> USART5_RX
- U1 pad 61: unconnected-(U1-PB8-Pad61) -> CAMERA_CTRL
- U1 pad 62: unconnected-(U1-PB9-Pad62) -> BEEPER
- U1 pad 8: unconnected-(U1-PC0-Pad8) -> ADC_VBAT
- U1 pad 9: unconnected-(U1-PC1-Pad9) -> ADC_CURR
Other:
- outline, holes or cut-outs redrawn

Commit message: Updated PCB Layout
Parts:
- added C47: 0.1uF, Capacitor_SMD:C_0402_1005Metric, F.Cu at (28.1, 31.0)
- added Q1: CSD17313Q2, Package_SON:Texas_DQK, B.Cu at (43.9, 48.2)
- added R29: 22R, Resistor_SMD:R_0402_1005Metric, B.Cu at (45.9, 48.5)
- added R30: 10K, Resistor_SMD:R_0402_1005Metric, B.Cu at (44.4, 50.0)
- added U8: SN74LV4T125RGYR, Library:VQFN-14_L3.5-W3.5-P0.50-BL-EP, F.Cu at (28.1, 33.8)
- C20: moved to B.Cu
- C21, IC2: moved to F.Cu
- moved S1 48.7 mm to (24.4, 51.8)
- moved L1 37.1 mm to (46.4, 46.0)
- moved R2 30.9 mm to (34.5, 52.5), turned to -90 degrees
- moved R3 28.8 mm to (35.5, 52.5), turned to -90 degrees
- moved C20 23.2 mm to (30.5, 42.9), turned to 90 degrees
- moved C30 22.9 mm to (37.6, 44.4)
- moved J5 18.7 mm to (46.4, 27.7)
- moved J1 13.7 mm to (30.2, 27.7)
- moved R16 11.8 mm to (34.9, 31.5), turned to 180 degrees
- moved C25 11.5 mm to (36.8, 31.5), turned to 0 degrees
- moved R15 11.2 mm to (38.7, 31.5), turned to 180 degrees
- moved R6 10.4 mm to (42.9, 34.3)
- moved R8 10.4 mm to (43.9, 34.3)
- moved R7 10.4 mm to (41.9, 34.3)
- moved C12 9.65 mm to (44.5, 32.0)
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Connections:
- J1 pad 4: UART5_RX -> USART5_RX
- J1 pad 5: MOTOR_1 -> MOTOR1_OUT
- J1 pad 6: MOTOR_2 -> MOTOR2_OUT
- J1 pad 7: MOTOR_3 -> MOTOR3_OUT
- J1 pad 8: MOTOR_4 -> MOTOR4_OUT
- J2 pad 1: VCC_10V -> VTX_VCC
- U1 pad 4: unconnected-(U1-PC15-Pad4) -> VTX_PW_SW
Other:
- board text added: "${REFERENCE}"

Commit message: Update PCB Layout
Parts:
- added C48: 1uF, Capacitor_SMD:C_0603_1608Metric, B.Cu at (46.3, 48.7)
- added C49: 10nF, Capacitor_SMD:C_0402_1005Metric, B.Cu at (43.8, 51.3)
- added C50: 2.2uF, Capacitor_SMD:C_0603_1608Metric, B.Cu at (41.2, 48.7)
- added D6: LED, LED_SMD:LED_0603_1608Metric, F.Cu at (51.2, 47.0)
- added IC5: LP2992IM5-3.3, Library:SOT95P280X145-5N, B.Cu at (43.8, 48.7)
- added J6: Conn_01x21_Pin, Library:Betaflight_Pad_F, F.Cu at (37.0, 27.0)
- added J8: Conn_01x20_Pin, Library:Betaflight_Pad_B, F.Cu at (37.1, 58.5)
- added Q2: SS8050, Package_TO_SOT_SMD:SOT-23, F.Cu at (23.6, 37.8)
- added R31: 1K, Resistor_SMD:R_0402_1005Metric, F.Cu at (23.5, 40.3)
- added R32: 100R, Resistor_SMD:R_0402_1005Metric, F.Cu at (53.8, 47.0)
- C25, R15, R16, U6: moved to F.Cu
- moved R16 9.51 mm to (44.4, 31.0), turned to 0 degrees
- moved S1 7.85 mm to (23.6, 44.0), turned to 90 degrees
- moved R29 6.68 mm to (52.5, 49.5)
- moved Q1 6.68 mm to (50.5, 49.2)
- moved R30 6.14 mm to (50.4, 51.0)
- moved C25 5.70 mm to (42.5, 31.0), turned to 180 degrees
- moved C47 4.83 mm to (28.2, 35.8), turned to 0 degrees
- moved U6 3.94 mm to (23.6, 51.5)
- moved R5 3.93 mm to (28.4, 52.5)
- moved C1 3.60 mm to (40.0, 52.5)
- moved L1 2.60 mm to (46.1, 43.5)
- moved C2 2.55 mm to (23.6, 48.3)
- moved C9 2.55 mm to (23.6, 47.2)
- moved R26 2.34 mm to (53.8, 52.5)
- moved D3 2.02 mm to (42.8, 43.9), turned to 90 degrees
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Connections:
- C11 pad 1: +5V -> VCC_IN
- C17 pad 1: +5V -> VCC_IN
- C20 pad 1: +5V -> VCC_IN
- C23 pad 1: VCC_5V_IN -> VCC_5V
- C24 pad 1: VCC_5V_IN -> VCC_5V
- IC3 pad 1: VCC_5V_IN -> VCC_5V
- IC3 pad 3: VCC_5V_IN -> VCC_5V
- IC4 pad 1: VCC_5V_IN -> VCC_5V
- IC4 pad 3: VCC_5V_IN -> VCC_5V
- J3 pad 5: I2C3_SDA -> I2C1_SDA
- J3 pad 6: I2C3_SCL -> I2C1_SCL
- R25 pad 2: +3.3V -> +3.3V_MCU
- R26 pad 2: +3.3V -> +3.3V_MCU
- R6 pad 1: BARO_SDA -> I2C1_SDA
- R7 pad 1: BARO_SCL -> I2C1_SCL
- S1 pad 2: +3.3V -> +3.3V_MCU
- U1 pad 39: LED_STRIP -> SERVO1
- U1 pad 40: I2C3_SDA -> SERVO2
- U1 pad 41: I2C3_SCL -> unconnected-(U1-PA8-Pad41)
- U1 pad 58: BARO_SCL -> I2C1_SCL
- U1 pad 59: BARO_SDA -> I2C1_SDA
- U2 pad 3: BARO_SDA -> I2C1_SDA
- U2 pad 4: BARO_SCL -> I2C1_SCL
- U3 pad 19: +5V -> VCC_IN
- U3 pad 21: +5V -> VCC_IN
- U3 pad 24: +5V -> VCC_IN
- U3 pad 3: +5V -> VCC_IN
Routing:
- net VCC_IN: track 0.00 -> 56.0 mm
- net VCC_5V: track 0.00 -> 27.8 mm
- net USB_DP: track 0.00 -> 23.5 mm, vias 0 -> 2
- net USB_DN: track 0.00 -> 23.4 mm, vias 0 -> 2
- net VBAT_IN: track 0.00 -> 17.2 mm, vias 0 -> 1
- net /Sensors/OSC_OUT: track 0.00 -> 11.7 mm
- net +3.3V_MCU: track 0.00 -> 10.1 mm
- net VCC_5V_USB: track 0.00 -> 9.56 mm, vias 0 -> 2
- net /Power/EN: track 0.00 -> 9.34 mm
- net USART1_RX: track 0.00 -> 8.54 mm, vias 0 -> 2
- net /Sensors/OSC_IN: track 0.00 -> 8.46 mm
- net +3.3VA_MCU: track 0.00 -> 7.66 mm
- net +3.3V_SENSOR: track 0.00 -> 5.24 mm
- net Net-(U2-SDO): track 0.00 -> 5.05 mm
- net /MCU_Core/VCAP_2: track 0.00 -> 4.82 mm
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- added copper zone on B.Cu, net Net-(U4-SW)
- added copper zone on B.Cu, net Net-(U5-SW)
- added copper zone on B.Cu, net VBAT_IN
- added copper zone on B.Cu, net VCC_10V
- added copper zone on B.Cu, net VCC_5V
Other:
- copper layers 2 -> 4
- board text added: "ACT"
- board text added: "PWR"
- board text added: "STA"

Commit message: Updated PCB Layout
Parts:
- moved C8 9.57 mm to (28.7, 37.2), turned to -90 degrees
- moved C4 9.47 mm to (27.7, 37.2), turned to -90 degrees
- moved C10 4.12 mm to (36.3, 32.0), turned to 90 degrees
- moved C19 3.73 mm to (34.2, 32.0), turned to 90 degrees
- moved C3 3.37 mm to (37.8, 34.5), turned to 90 degrees
- moved C18 3.33 mm to (35.3, 32.0), turned to 90 degrees
- moved D5 2.79 mm to (51.2, 49.7)
- moved D4 2.79 mm to (51.2, 52.5)
- moved R26 2.79 mm to (53.8, 49.7)
- moved R25 2.79 mm to (53.8, 52.5)
- moved IC1 1.76 mm to (35.3, 34.5), turned to 180 degrees
- moved R2 0.19 mm to (34.5, 52.7)
- moved R3 0.19 mm to (35.6, 52.7)
- turned S1 to -90 degrees
Connections:
- J6 pad 7: VBAT_IN -> VBAT
- J8 pad 11: I2C1_SDA -> I2C1_SCL
- J8 pad 12: I2C1_SCL -> I2C1_SDA
- U1 pad 41: unconnected-(U1-PA8-Pad41) -> LED_STRIP
- U8 pad 2: MOTOR1 -> MOTOR2
- U8 pad 3: MOTOR1_OUT -> MOTOR2_OUT
- U8 pad 5: MOTOR2 -> MOTOR1
- U8 pad 6: MOTOR2_OUT -> MOTOR1_OUT
Routing:
- net I2C1_SDA: track 1.72 -> 46.4 mm, vias 0 -> 4
- net I2C1_SCL: track 1.56 -> 44.0 mm, vias 0 -> 4
- net LED_STRIP: track 0.00 -> 42.2 mm, vias 0 -> 2
- net VCC_IN: track 56.0 -> 14.2 mm
- net SERVO2: track 0.00 -> 38.2 mm, vias 0 -> 2
- net CAMERA_CTRL: track 0.00 -> 37.1 mm, vias 0 -> 4
- net ADC_RSSI: track 0.00 -> 32.2 mm, vias 0 -> 2
- net ADC_CURR: track 0.00 -> 31.6 mm, vias 0 -> 3
- net USART4_RX: track 0.00 -> 31.4 mm, vias 0 -> 4
- net USART6_TX: track 0.00 -> 30.8 mm, vias 0 -> 3
- net USART4_TX: track 0.00 -> 30.2 mm, vias 0 -> 4
- net SERVO1: track 0.00 -> 30.0 mm, vias 0 -> 2
- net SPI2_SCK: track 0.00 -> 30.0 mm, vias 0 -> 2
- net USART6_RX: track 0.00 -> 26.7 mm, vias 0 -> 3
- net BEEPER-: track 0.00 -> 26.2 mm, vias 0 -> 2
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
Commit message: Finished PCB V1.0
Parts:
- removed Q1: CSD17313Q2, Package_SON:Texas_DQK
- removed R29: 22R, Resistor_SMD:R_0402_1005Metric
- removed R30: 10K, Resistor_SMD:R_0402_1005Metric
- added G***: LOGO, Library:NekoPurrTech_logo, F.Cu at (50.3, 32.1)
- added G***: LOGO, Library:skylark_logo, F.Cu at (27.8, 51.6)
- moved R8 2.57 mm to (41.5, 35.3)
- moved R6 0.50 mm to (43.5, 35.3)
- moved R7 0.50 mm to (42.5, 35.3)
- turned C17 to -90 degrees
Connections:
- C23 pad 1: VCC_5V -> VCC_IN
- C24 pad 1: VCC_5V -> VCC_IN
- C48 pad 1: VCC_5V -> VCC_IN
- C50 pad 1: +3.3V_SENSOR -> +3.3V_PREP
- IC3 pad 1: VCC_5V -> VCC_IN
- IC3 pad 3: VCC_5V -> VCC_IN
- IC4 pad 1: VCC_5V -> VCC_IN
- IC4 pad 3: VCC_5V -> VCC_IN
- IC5 pad 1: VCC_5V -> VCC_IN
- IC5 pad 3: VCC_5V -> VCC_IN
- IC5 pad 5: +3.3V_SENSOR -> +3.3V_PREP
- J2 pad 1: VTX_VCC -> VCC_10V
- J3 pad 1: VCC_5V -> VCC_IN
- J4 pad 1: VCC_5V -> VCC_IN
- J5 pad 1: unconnected-(J5-Pin_1-Pad1) -> VCC_IN
- J5 pad 2: unconnected-(J5-Pin_2-Pad2) -> GND
- J5 pad 3: unconnected-(J5-Pin_3-Pad3) -> VRX
- J5 pad MP: unconnected-(J5-MountPin-PadMP) -> GND
- J6 pad 12: unconnected-(J6-Pin_12-Pad12) -> USART2_RX
- J6 pad 13: unconnected-(J6-Pin_13-Pad13) -> USART2_TX
- J8 pad 10: +3.3V_MCU -> +3.3V_PREP
- J8 pad 14: VTX_VCC -> VCC_10V
- R17 pad 1: /Power/EN -> /Power/EN1
- R22 pad 1: /Power/EN -> /Power/EN2
- U4 pad 3: /Power/EN -> /Power/EN1
- U5 pad 3: /Power/EN -> /Power/EN2
- U6 pad 5: VCC_5V -> VCC_IN
Routing:
- net VCC_IN: track 14.2 -> 163.3 mm, vias 0 -> 6
- net +3.3V_MCU: track 32.1 -> 143.7 mm, vias 0 -> 12
- net VCC_10V: track 0.00 -> 64.3 mm, vias 0 -> 4
- net +3.3V_SENSOR: track 10.6 -> 65.5 mm, vias 0 -> 4
- net USART5_RX: track 0.00 -> 42.2 mm, vias 0 -> 4
- net USART2_RX: track 22.7 -> 57.2 mm, vias 2 -> 4
- net VRX: track 24.0 -> 53.9 mm, vias 3 -> 4
- net USART2_TX: track 20.2 -> 48.3 mm, vias 2 -> 4
- net VTX: track 0.00 -> 21.1 mm, vias 0 -> 2
- net +3.3V_PREP: track 0.00 -> 16.7 mm, vias 0 -> 2
- net VBAT: track 5.91 -> 21.7 mm, vias 1 -> 2
- net VCC_5V: track 31.4 -> 20.6 mm, vias 0 -> 2
- net /Power/EN: track 9.34 -> 0.00 mm
- net Net-(U5-SW): track 0.00 -> 9.02 mm, vias 0 -> 2
- net Net-(U4-SW): track 0.00 -> 7.80 mm, vias 0 -> 2
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- added copper zone on B.Cu, net GND
- added copper zone on F.Cu, net GND
- added copper zone on In1.Cu, net GND
- added copper zone on In2.Cu, net GND
Other:
- board text added: "3V3"
- board text added: "5V"
- board text added: "9V"
- board text added: "B+"
- board text added: "B-"
- board text added: "BAT"
- board text added: "CAM"
- board text added: "CC"
- board text added: "CL"
- board text added: "DA"
- board text added: "FLASH"
- board text added: "G"
- board text added: "LED"
- board text added: "MCU"
- board text added: "R2"
- board text added: "R3"
- board text added: "R4"
- board text added: "R6"
- board text added: "RS"
- board text added: "S1"
- board text added: "S2"
- board text added: "SBUS"
- board text added: "SENSORS"
- board text added: "SkyLark V1.0"
- board text added: "T2"
- board text added: "T3"
- board text added: "T4"
- board text added: "T6"
- board text added: "USB"
- board text added: "VTX"
